File: board/flashlight-boost.brd (EAGLE design)
At the start: 15 x 25 mm, 9 parts

Commit message: Fixing voltage divider.
The voltage divider was setup to yield a control voltage of 0.6v which for a 2.4v input sets up the LED driver for a driver current of just over 25mA.  The drive current should be between 80mA and 100mA.  Lowering R1 in the divider to somewhere between 178k and 150k will do just that.
Parts:
- R2: value 300k -> 150k
Changed lines of the file:
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@@
 <element name="LED-1" library="wirepad" package="2,54/1,0" value="GND" x="13.335" y="1.905"/>
 <element name="U$1" library="Synapseware" package="NSOIC-8" value="LTC3490NSOIC-8" x="7.62" y="12.7" rot="R180"/>
-<element name="R2" library="SparkFun-Resistors" package="0603-RES" value="300k" x="12.065" y="14.986" rot="R90"/>
+<element name="R2" library="SparkFun-Resistors" package="0603-RES" value="150k" x="12.065" y="14.986" rot="R90"/>
 <element name="R3" library="SparkFun-Resistors" package="0603-RES" value="100k" x="12.065" y="10.16" rot="R90"/>
 <element name="C1" library="SparkFun-Passives" package="1206" value="4.7uF/XR7" x="8.89" y="5.715"/>
